File: tests/fixtures/Arduino_Mega/Arduino_Mega.kicad_sch (KiCad schematic)
At the start: 7 parts, among them J1 Power, J2 PWM, J3 Analog, J4 PWM, J5 Analog, J6 Communication, J7 Digital

Commit message: chore: add Phase 9 (GRPO Spatial Reasoning Training) to roadmap
Phase 9 covers DeepSeek-style RL training with coordinate-grounded
reward signals on synthetic PCB maze data. Includes GRPO-01 through
GRPO-07 requirements and 4 planned sub-plans.

Generated with [Claude Code](https://claude.ai/code)
via [Happy](https://happy.engineering)

Co-Authored-By: Claude <noreply@anthropic.com>
Co-Authored-By: Happy <yesreply@happy.engineering>
Parts:
- added R? (x4): (no value), symbol Device:R_Small_US
Connections:
- net +3V3: no longer J1.4 (Pin_4)
- net +5V: no longer J1.5 (Pin_5)
- net GND: no longer J1.6 (Pin_6), J1.7 (Pin_7)
- net IOREF: no longer J1.2 (Pin_2)
- net VCC: no longer J1.8 (Pin_8)
- net ~{RESET}: no longer J1.3 (Pin_3)
Other:
- moved on the sheet: J1
Changed lines of the file:
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@@
     (effects (font (size 1.27 1.27)) (justify right bottom))
   )
-  (symbol (lib_id "Connector_Generic:Conn_01x08") (at 39.37 39.37 0) (unit 1)
+  (symbol (lib_id "Connector_Generic:Conn_01x08") (at 50 30) (unit 1)
     (in_bom yes) (on_board yes) (dnp no)
     (property "Reference" "J1" (at 39.37 29.21 0)
@@
     )
   )
+  (symbol (lib_name "Device:R_Small_US") (lib_id "Device:R_Small_US") (at 50 30)
+    (in_bom yes) (on_board yes)
+    (property "Reference" "R?" (id 0) (at 0 0)
+      (effects (font (size 1.27 1.27)))
+    )
+    (property "Value" "" (id 1) (at 0 0)
+      (effects (font (size 1.27 1.27)))
+    )
+    (property "Footprint" "" (id 2) (at 0 0)
+      (effects (font (size 1.27 1.27)) hide)
+    )
+    (property "Datasheet" "~" (id 3) (at 0 0)
+      (effects (font (size 1.27 1.27)) hide)
+    )
+  )
+  (symbol (lib_name "Device:R_Small_US") (lib_id "Device:R_Small_US") (at 50 30)
+    (in_bom yes) (on_board yes)
+    (property "Reference" "R?" (id 0) (at 0 0)
+      (effects (font (size 1.27 1.27)))
+    )
+    (property "Value" "" (id 1) (at 0 0)
+      (effects (font (size 1.27 1.27)))
+    )
+    (property "Footprint" "" (id 2) (at 0 0)
+      (effects (font (size 1.27 1.27)) hide)
+    )
+    (property "Datasheet" "~" (id 3) (at 0 0)
+      (effects (font (size 1.27 1.27)) hide)
+    )
+  )
+  (symbol (lib_name "Device:R_Small_US") (lib_id "Device:R_Small_US") (at 50 30)
+    (in_bom yes) (on_board yes)
+    (property "Reference" "R?" (id 0) (at 0 0)
+      (effects (font (size 1.27 1.27)))
+    )
+    (property "Value" "" (id 1) (at 0 0)
+      (effects (font (size 1.27 1.27)))
+    )
+    (property "Footprint" "" (id 2) (at 0 0)
+      (effects (font (size 1.27 1.27)) hide)
+    )
+    (property "Datasheet" "~" (id 3) (at 0 0)
+      (effects (font (size 1.27 1.27)) hide)
+    )
+  )
+  (symbol (lib_name "Device:R_Small_US") (lib_id "Device:R_Small_US") (at 50 30)
+    (in_bom yes) (on_board yes)
+    (property "Reference" "R?" (id 0) (at 0 0)
+      (effects (font (size 1.27 1.27)))
+    )
+    (property "Value" "" (id 1) (at 0 0)
+      (effects (font (size 1.27 1.27)))
+    )
+    (property "Footprint" "" (id 2) (at 0 0)
+      (effects (font (size 1.27 1.27)) hide)
+    )
+    (property "Datasheet" "~" (id 3) (at 0 0)
+      (effects (font (size 1.27 1.27)) hide)
+    )
+  )
