File: tests/fixtures/Arduino_Mega/Arduino_Mega.kicad_sch (KiCad schematic)
At the start: 40 parts, among them J1 Power, J2 PWM, J3 Analog, J4 PWM, J5 Analog, J6 Communication, J7 Digital

Commit message: feat: add schematic validation pipeline with 7 pre-flight checks
Built across 3 sessions fixing code-generated KiCad backplane schematics.
Every check addresses a systematic failure mode discovered in production.

New checks:
- format_check: 9 KiCad 10 S-expression format rules (no ;;, no tabs, etc.)
- symbol_resolution: lib_id → definition resolution chain (embedded → project → global)
- grid_check: pin/wire off-grid detection (prevents silent connection failures)
- symbol_mismatch: embedded vs library copy divergence detection
- Bare lib_id detection (flags Library:Symbol format violations)

New operation: validate_schematic (combines all checks + power + annotation)

Also fixes MIN_KICAD_VERSION constant (was v6, docstring said v7).

Generated with [Claude Code](https://claude.ai/code)
via [Happy](https://happy.engineering)

Co-Authored-By: Claude <noreply@anthropic.com>
Co-Authored-By: Happy <yesreply@happy.engineering>
Parts:
- added R? (x5): (no value), symbol Device:R_Small_US
Other:
- moved on the sheet: J1
Changed lines of the file:
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@@
     (effects (font (size 1.27 1.27)) (justify right bottom))
   )
-  (symbol (lib_id "Connector_Generic:Conn_01x08") (at 50 30) (unit 1)
+  (symbol (lib_id "Connector_Generic:Conn_01x08") (at 100 200) (unit 1)
     (in_bom yes) (on_board yes) (dnp no)
     (property "Reference" "J1" (at 39.37 29.21 0)
@@
     )
   )
+  (symbol (lib_name "Device:R_Small_US") (lib_id "Device:R_Small_US") (at 50 30)
+    (in_bom yes) (on_board yes)
+    (property "Reference" "R?" (id 0) (at 0 0)
+      (effects (font (size 1.27 1.27)))
+    )
+    (property "Value" "" (id 1) (at 0 0)
+      (effects (font (size 1.27 1.27)))
+    )
+    (property "Footprint" "" (id 2) (at 0 0)
+      (effects (font (size 1.27 1.27)) hide)
+    )
+    (property "Datasheet" "~" (id 3) (at 0 0)
+      (effects (font (size 1.27 1.27)) hide)
+    )
+  )
+  (symbol (lib_name "Device:R_Small_US") (lib_id "Device:R_Small_US") (at 50 30)
+    (in_bom yes) (on_board yes)
+    (property "Reference" "R?" (id 0) (at 0 0)
+      (effects (font (size 1.27 1.27)))
+    )
+    (property "Value" "" (id 1) (at 0 0)
+      (effects (font (size 1.27 1.27)))
+    )
+    (property "Footprint" "" (id 2) (at 0 0)
+      (effects (font (size 1.27 1.27)) hide)
+    )
+    (property "Datasheet" "~" (id 3) (at 0 0)
+      (effects (font (size 1.27 1.27)) hide)
+    )
+  )
+  (symbol (lib_name "Device:R_Small_US") (lib_id "Device:R_Small_US") (at 50 30)
+    (in_bom yes) (on_board yes)
+    (property "Reference" "R?" (id 0) (at 0 0)
+      (effects (font (size 1.27 1.27)))
+    )
+    (property "Value" "" (id 1) (at 0 0)
+      (effects (font (size 1.27 1.27)))
+    )
+    (property "Footprint" "" (id 2) (at 0 0)
+      (effects (font (size 1.27 1.27)) hide)
+    )
+    (property "Datasheet" "~" (id 3) (at 0 0)
+      (effects (font (size 1.27 1.27)) hide)
+    )
+  )
+  (symbol (lib_name "Device:R_Small_US") (lib_id "Device:R_Small_US") (at 50 30)
+    (in_bom yes) (on_board yes)
+    (property "Reference" "R?" (id 0) (at 0 0)
+      (effects (font (size 1.27 1.27)))
+    )
+    (property "Value" "" (id 1) (at 0 0)
+      (effects (font (size 1.27 1.27)))
+    )
+    (property "Footprint" "" (id 2) (at 0 0)
+      (effects (font (size 1.27 1.27)) hide)
+    )
+    (property "Datasheet" "~" (id 3) (at 0 0)
+      (effects (font (size 1.27 1.27)) hide)
+    )
+  )
+  (symbol (lib_name "Device:R_Small_US") (lib_id "Device:R_Small_US") (at 50 30)
+    (in_bom yes) (on_board yes)
+    (property "Reference" "R?" (id 0) (at 0 0)
+      (effects (font (size 1.27 1.27)))
+    )
+    (property "Value" "" (id 1) (at 0 0)
+      (effects (font (size 1.27 1.27)))
+    )
+    (property "Footprint" "" (id 2) (at 0 0)
+      (effects (font (size 1.27 1.27)) hide)
+    )
+    (property "Datasheet" "~" (id 3) (at 0 0)
+      (effects (font (size 1.27 1.27)) hide)
+    )
+  )

Commit message: chore: update Arduino_Mega fixture for v3.0 spatial/DFM tests
Generated with [Claude Code](https://claude.ai/code)
via [Happy](https://happy.engineering)

Co-Authored-By: Claude <noreply@anthropic.com>
Co-Authored-By: Happy <yesreply@happy.engineering>
Parts:
- added R? (x46): (no value), symbol Device:R_Small_US
Other:
- moved on the sheet: J1

Commit message: fix(erc-auto-fix): persist in-memory mutations to disk before verification
ERC auto-fix was running post-repair verification against stale disk
content because in-memory IR mutations were never written back. Added
schematic.to_file() calls after each repair and after rollback restore.
Also fixed hierarchical sheet_filter logic for sub-sheets.

Generated with [Claude Code](https://claude.ai/code)
via [Happy](https://happy.engineering)

Co-Authored-By: Claude <noreply@anthropic.com>
Co-Authored-By: Happy <yesreply@happy.engineering>
Parts:
- added R? (x4): (no value), symbol Device:R_Small_US
Changed lines of the file:
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@@
     (effects (font (size 1.27 1.27)) (justify right bottom))
   )
-  (symbol (lib_id "Connector_Generic:Conn_01x08") (at 50 30) (unit 1)
+  (symbol (lib_id "Connector_Generic:Conn_01x08") (at 50.0 30.0) (unit 1)
     (in_bom yes) (on_board yes) (dnp no)
     (property "Reference" "J1" (at 39.37 29.21 0)
@@
     )
   )
+  (symbol (lib_name "Device:R_Small_US") (lib_id "Device:R_Small_US") (at 50 30)
+    (in_bom yes) (on_board yes)
+    (property "Reference" "R?" (id 0) (at 0 0)
+      (effects (font (size 1.27 1.27)))
+    )
+    (property "Value" "" (id 1) (at 0 0)
+      (effects (font (size 1.27 1.27)))
+    )
+    (property "Footprint" "" (id 2) (at 0 0)
+      (effects (font (size 1.27 1.27)) hide)
+    )
+    (property "Datasheet" "~" (id 3) (at 0 0)
+      (effects (font (size 1.27 1.27)) hide)
+    )
+  )
+  (symbol (lib_name "Device:R_Small_US") (lib_id "Device:R_Small_US") (at 50 30)
+    (in_bom yes) (on_board yes)
+    (property "Reference" "R?" (id 0) (at 0 0)
+      (effects (font (size 1.27 1.27)))
+    )
+    (property "Value" "" (id 1) (at 0 0)
+      (effects (font (size 1.27 1.27)))
+    )
+    (property "Footprint" "" (id 2) (at 0 0)
+      (effects (font (size 1.27 1.27)) hide)
+    )
+    (property "Datasheet" "~" (id 3) (at 0 0)
+      (effects (font (size 1.27 1.27)) hide)
+    )
+  )
+  (symbol (lib_name "Device:R_Small_US") (lib_id "Device:R_Small_US") (at 50 30)
+    (in_bom yes) (on_board yes)
+    (property "Reference" "R?" (id 0) (at 0 0)
+      (effects (font (size 1.27 1.27)))
+    )
+    (property "Value" "" (id 1) (at 0 0)
+      (effects (font (size 1.27 1.27)))
+    )
+    (property "Footprint" "" (id 2) (at 0 0)
+      (effects (font (size 1.27 1.27)) hide)
+    )
+    (property "Datasheet" "~" (id 3) (at 0 0)
+      (effects (font (size 1.27 1.27)) hide)
+    )
+  )
+  (symbol (lib_name "Device:R_Small_US") (lib_id "Device:R_Small_US") (at 50 30)
+    (in_bom yes) (on_board yes)
+    (property "Reference" "R?" (id 0) (at 0 0)
+      (effects (font (size 1.27 1.27)))
+    )
+    (property "Value" "" (id 1) (at 0 0)
+      (effects (font (size 1.27 1.27)))
+    )
+    (property "Footprint" "" (id 2) (at 0 0)
+      (effects (font (size 1.27 1.27)) hide)
+    )
+    (property "Datasheet" "~" (id 3) (at 0 0)
+      (effects (font (size 1.27 1.27)) hide)
+    )
+  )

Commit message: fix: kiutils serialization defects (#11, #12) and topology-aware snap_to_grid (#1, #5)
- Add _fix_kiutils_output() post-processor to fix kiutils 1.4.8 bugs:
  quotes generator value, injects generator_version, adds rotation to
  no_connect (at ...) expressions so kicad-cli accepts files
- Set angle=0 on NoConnect Position in schematic_ir.py for IR correctness
- Rewrite snap_to_grid() with union-find clustering replacing rounding-based
  endpoint grouping — preserves wire connectivity within SNAP_TOLERANCE
- Add tests for union-find snap_to_grid and Arduino_Mega fixture updates

Closes #1, #2, #3, #4, #5, #6, #10, #11, #12

Generated with [Claude Code](https://claude.ai/code)
via [Happy](https://happy.engineering)

Co-Authored-By: Claude <noreply@anthropic.com>
Co-Authored-By: Happy <yesreply@happy.engineering>
Parts:
- added R? (x12): (no value), symbol Device:R_Small_US
Changed lines of the file:
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@@
-(kicad_sch (version 20250114) (generator eeschema)
+(kicad_sch (version 20250114) (generator "eeschema")
+  (generator_version "10.0")
   (paper "A4")
   (title_block
@@
   (junction (at 74.93 119.38) (diameter 0) (color 0 0 0 0)
   )
-  (no_connect (at 34.29 31.75))
+  (no_connect (at 34.29 31.75 0))
   (wire (pts (xy 62.23 77.47) (xy 74.93 77.47))
     (stroke (width 0) (type solid))
@@
     (effects (font (size 1.27 1.27)) (justify right bottom))
   )
-  (symbol (lib_id "Connector_Generic:Conn_01x08") (at 50.0 30.0) (unit 1)
+  (symbol (lib_id "Connector_Generic:Conn_01x08") (at 50 30) (unit 1)
     (in_bom yes) (on_board yes) (dnp no)
     (property "Reference" "J1" (at 39.37 29.21 0)
@@
     )
   )
+  (symbol (lib_name "Device:R_Small_US") (lib_id "Device:R_Small_US") (at 50 30)
+    (in_bom yes) (on_board yes)
+    (property "Reference" "R?" (id 0) (at 0 0)
+      (effects (font (size 1.27 1.27)))
+    )
+    (property "Value" "" (id 1) (at 0 0)
+      (effects (font (size 1.27 1.27)))
+    )
+    (property "Footprint" "" (id 2) (at 0 0)
+      (effects (font (size 1.27 1.27)) hide)
+    )
+    (property "Datasheet" "~" (id 3) (at 0 0)
+      (effects (font (size 1.27 1.27)) hide)
+    )
+  )
+  (symbol (lib_name "Device:R_Small_US") (lib_id "Device:R_Small_US") (at 50 30)
+    (in_bom yes) (on_board yes)
+    (property "Reference" "R?" (id 0) (at 0 0)
+      (effects (font (size 1.27 1.27)))
+    )
+    (property "Value" "" (id 1) (at 0 0)
+      (effects (font (size 1.27 1.27)))
+    )
+    (property "Footprint" "" (id 2) (at 0 0)
+      (effects (font (size 1.27 1.27)) hide)
+    )
+    (property "Datasheet" "~" (id 3) (at 0 0)
+      (effects (font (size 1.27 1.27)) hide)
+    )
+  )
+  (symbol (lib_name "Device:R_Small_US") (lib_id "Device:R_Small_US") (at 50 30)
+    (in_bom yes) (on_board yes)
+    (property "Reference" "R?" (id 0) (at 0 0)
+      (effects (font (size 1.27 1.27)))
+    )
+    (property "Value" "" (id 1) (at 0 0)
+      (effects (font (size 1.27 1.27)))
+    )
+    (property "Footprint" "" (id 2) (at 0 0)
+      (effects (font (size 1.27 1.27)) hide)
+    )
+    (property "Datasheet" "~" (id 3) (at 0 0)
+      (effects (font (size 1.27 1.27)) hide)
+    )
+  )
+  (symbol (lib_name "Device:R_Small_US") (lib_id "Device:R_Small_US") (at 50 30)
+    (in_bom yes) (on_board yes)
+    (property "Reference" "R?" (id 0) (at 0 0)
+      (effects (font (size 1.27 1.27)))
+    )
+    (property "Value" "" (id 1) (at 0 0)
+      (effects (font (size 1.27 1.27)))
+    )
+    (property "Footprint" "" (id 2) (at 0 0)
+      (effects (font (size 1.27 1.27)) hide)
+    )
+    (property "Datasheet" "~" (id 3) (at 0 0)
+      (effects (font (size 1.27 1.27)) hide)
+    )
+  )
+  (symbol (lib_name "Device:R_Small_US") (lib_id "Device:R_Small_US") (at 50 30)
+    (in_bom yes) (on_board yes)
+    (property "Reference" "R?" (id 0) (at 0 0)
+      (effects (font (size 1.27 1.27)))
+    )
+    (property "Value" "" (id 1) (at 0 0)
+      (effects (font (size 1.27 1.27)))
+    )
+    (property "Footprint" "" (id 2) (at 0 0)
+      (effects (font (size 1.27 1.27)) hide)
+    )
+    (property "Datasheet" "~" (id 3) (at 0 0)
+      (effects (font (size 1.27 1.27)) hide)
+    )
+  )
+  (symbol (lib_name "Device:R_Small_US") (lib_id "Device:R_Small_US") (at 50 30)
+    (in_bom yes) (on_board yes)
+    (property "Reference" "R?" (id 0) (at 0 0)
+      (effects (font (size 1.27 1.27)))
+    )
+    (property "Value" "" (id 1) (at 0 0)
+      (effects (font (size 1.27 1.27)))
+    )
+    (property "Footprint" "" (id 2) (at 0 0)
+      (effects (font (size 1.27 1.27)) hide)
+    )
+    (property "Datasheet" "~" (id 3) (at 0 0)
+      (effects (font (size 1.27 1.27)) hide)
+    )
+  )
+  (symbol (lib_name "Device:R_Small_US") (lib_id "Device:R_Small_US") (at 50 30)
+    (in_bom yes) (on_board yes)
+    (property "Reference" "R?" (id 0) (at 0 0)
+      (effects (font (size 1.27 1.27)))
+    )
+    (property "Value" "" (id 1) (at 0 0)
+      (effects (font (size 1.27 1.27)))
+    )
+    (property "Footprint" "" (id 2) (at 0 0)
+      (effects (font (size 1.27 1.27)) hide)
+    )
+    (property "Datasheet" "~" (id 3) (at 0 0)
+      (effects (font (size 1.27 1.27)) hide)
+    )
+  )
+  (symbol (lib_name "Device:R_Small_US") (lib_id "Device:R_Small_US") (at 50 30)
+    (in_bom yes) (on_board yes)
+    (property "Reference" "R?" (id 0) (at 0 0)
+      (effects (font (size 1.27 1.27)))
+    )
+    (property "Value" "" (id 1) (at 0 0)
+      (effects (font (size 1.27 1.27)))
+    )
+    (property "Footprint" "" (id 2) (at 0 0)
+      (effects (font (size 1.27 1.27)) hide)
+    )
+    (property "Datasheet" "~" (id 3) (at 0 0)
+      (effects (font (size 1.27 1.27)) hide)
+    )
+  )
+  (symbol (lib_name "Device:R_Small_US") (lib_id "Device:R_Small_US") (at 50 30)
+    (in_bom yes) (on_board yes)
+    (property "Reference" "R?" (id 0) (at 0 0)
+      (effects (font (size 1.27 1.27)))
+    )
+    (property "Value" "" (id 1) (at 0 0)
+      (effects (font (size 1.27 1.27)))
+    )
+    (property "Footprint" "" (id 2) (at 0 0)
+      (effects (font (size 1.27 1.27)) hide)
+    )
+    (property "Datasheet" "~" (id 3) (at 0 0)
+      (effects (font (size 1.27 1.27)) hide)
+    )
+  )
+  (symbol (lib_name "Device:R_Small_US") (lib_id "Device:R_Small_US") (at 50 30)
+    (in_bom yes) (on_board yes)
+    (property "Reference" "R?" (id 0) (at 0 0)
+      (effects (font (size 1.27 1.27)))
+    )
+    (property "Value" "" (id 1) (at 0 0)
+      (effects (font (size 1.27 1.27)))
+    )
+    (property "Footprint" "" (id 2) (at 0 0)
+      (effects (font (size 1.27 1.27)) hide)
+    )
+    (property "Datasheet" "~" (id 3) (at 0 0)
+      (effects (font (size 1.27 1.27)) hide)
+    )
+  )
+  (symbol (lib_name "Device:R_Small_US") (lib_id "Device:R_Small_US") (at 50 30)
+    (in_bom yes) (on_board yes)
+    (property "Reference" "R?" (id 0) (at 0 0)
+      (effects (font (size 1.27 1.27)))
+    )
+    (property "Value" "" (id 1) (at 0 0)
+      (effects (font (size 1.27 1.27)))
+    )
+    (property "Footprint" "" (id 2) (at 0 0)
+      (effects (font (size 1.27 1.27)) hide)
+    )
+    (property "Datasheet" "~" (id 3) (at 0 0)
+      (effects (font (size 1.27 1.27)) hide)
+    )
+  )
+  (symbol (lib_name "Device:R_Small_US") (lib_id "Device:R_Small_US") (at 50 30)
+    (in_bom yes) (on_board yes)
+    (property "Reference" "R?" (id 0) (at 0 0)
+      (effects (font (size 1.27 1.27)))
+    )
+    (property "Value" "" (id 1) (at 0 0)
+      (effects (font (size 1.27 1.27)))
+    )
+    (property "Footprint" "" (id 2) (at 0 0)
+      (effects (font (size 1.27 1.27)) hide)
+    )
+    (property "Datasheet" "~" (id 3) (at 0 0)
+      (effects (font (size 1.27 1.27)) hide)
+    )
+  )

Commit message: feat: add 4 advanced PCB operations (#44-#47), pre-analysis, multi-pass routing
New operations (94→98):
- #44 route_diff_pair: impedance-controlled differential pair routing
- #45 match_lengths: serpentine tuning for net pair length matching
- #46 analyze_split_plane: split plane boundary crossing detection (read-only)
- #47 fix_silkscreen_over_copper: auto-reposition ref designators

New modules:
- pre_analysis.py: overlap/collision detection before operation execution
- multi_pass.py: 3-pass routing strategy (rip-up, aggressive, final)
- pcb_netlist.py: netlist extraction from PCB native parser
- silkscreen_clearance.py: silkscreen-copper overlap detection engine

Infrastructure:
- PcbIR native parser integration, net_id_map extraction
- ExtractedRoute for route path extraction from PCB segments
- 74 new tests across 4 feature test files

Generated with [Claude Code](https://claude.ai/code)
via [Happy](https://happy.engineering)

Co-Authored-By: Claude <noreply@anthropic.com>
Co-Authored-By: Happy <yesreply@happy.engineering>
Parts:
- added R? (x29): (no value), symbol Device:R_Small_US
- J1, J2, J3, J4, J5, J6, J7, R? (x100): now left out of the parts list
Other:
- moved on the sheet: J1
