File: tests/fixtures/smd_test_board.kicad_pcb (KiCad board)
At the start: 1 copper layers, 50 x 30 mm, 8 parts

Commit message: test(99-03): add sc-3 e2e drc and sc-5 45-vs-manhattan tests
Add two slow integration tests proving Phase 99-01/99-02 work survives
a real Freerouting to kicad-cli DRC round-trip.

Six Rule 1/3 fixes required to make SC-3 pass (blocking issues):
- dsn_generator: fix doubled default class header on empty member set
- dsn_generator: take copper token from SMD pad layer set (no spaces)
- freerouting: fix extract_pcb_net_names for KiCad 10 net form
- freerouting: fix SES resolution divisor (1000 not 10000)
- freerouting: remove wrong Y-negation (KiCad Y-down preserved)
- FreerouteBatch.java: add snap_angle arg with preferred directions

Fix smd_test_board fixture (was unloadable by kicad-cli): move net
declarations to top level, add missing B.Cu layer, fix layer numbers.

Update test_phase99_ses_r6_multilayer.py assertions for the resolution
and Y-negation corrections.

SC-5 marked xfail on Freerouting v2.2.4 (batch autorouter ignores DSN
snap_angle directive; workaround does not beat default any-angle mode).

All 42 Phase 99 unit tests pass. 307 routing/parser tests pass.
Other:
- copper layers 1 -> 2
Changed lines of the file:
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@@
 	(layers
 		(0 "F.Cu" signal)
+		(2 "B.Cu" signal)
+		(13 "F.Paste" user)
+		(15 "B.Paste" user)
+		(5 "F.SilkS" user "F.Silkscreen")
+		(7 "B.SilkS" user "B.Silkscreen")
+		(1 "F.Mask" user)
+		(3 "B.Mask" user)
+		(25 "Edge.Cuts" user)
 		(31 "F.CrtYd" user "F.Courtyard")
-		(32 "B.CrtYd" user "B.Courtyard")
+		(29 "B.CrtYd" user "B.Courtyard")
+		(35 "F.Fab" user)
 		(33 "B.Fab" user)
-		(35 "F.Fab" user)
-		(36 "B.SilkS" user "B.Silkscreen")
-		(37 "F.SilkS" user "F.Silkscreen")
-		(38 "B.Mask" user)
-		(39 "F.Mask" user)
-		(40 "B.Paste" user)
-		(41 "F.Paste" user)
-		(44 "Edge.Cuts" user)
 	)
 	(setup
@@
 			(outputdirectory "")
 		)
-		(net 0 "")
-		(net 1 "NET_A")
-		(net 2 "NET_B")
-		(net 3 "NET_C")
-		(net 4 "NET_D")
-		(net 5 "NET_E")
-		(net 6 "NET_F")
-		(net 7 "VCC")
-		(net 8 "GND")
 	)
+	(net 0 "")
+	(net 1 "NET_A")
+	(net 2 "NET_B")
+	(net 3 "NET_C")
+	(net 4 "NET_D")
+	(net 5 "NET_E")
+	(net 6 "NET_F")
+	(net 7 "VCC")
+	(net 8 "GND")
 	(segment
 		(start 5 5)
